Commit message: create srdf on the go

File: config/srdf/pal_sea_arm.srdf.xacro (robot description, xacro)
@@ -1,19 +1,36 @@
-<?xml version="1.0" ?>
+<?xml version="1.0"?>
 <!--This does not replace URDF, and is not an extension of URDF.
     This is a format for representing semantic information about the robot structure.
-    A URDF file must exist for this robot as well, where the joints and the links that are referenced are defined
+    A URDF file must exist for this robot as well, where the joints and the links that are referenced
+are defined
 -->
-<robot name="pal_sea_arm" xmlns:xacro="http://ros.org/wiki/xacro">
-    <xacro:arg name="end_effector" default="pal-pro-gripper"/>
-    <xacro:arg name="ft_sensor" default="false"/>
-    <xacro:property name="end_effector" value="$(arg end_effector)"/>
-    <xacro:property name="ft_sensor" value="$(arg ft_sensor)"/>
-    <xacro:property name="has_ft_sensor" value="${ft_sensor not in ['false', False]}"/>
-    <xacro:property name="robot" value="pal_sea_arm"/>
-    <!--GROUPS: Representation of a set of joints and links. This can be useful for specifying DOF to plan for, defining arms, end effectors, etc-->
-    <!--LINKS: When a link is specified, the parent joint of that link (if it exists) is automatically included-->
-    <!--JOINTS: When a joint is specified, the child link of that joint (which will always exist) is automatically included-->
-    <!--CHAINS: When a chain is specified, all the links along the chain (including endpoints) are included in the group. Additionally, all the joints that are parents to included links are also included. This means that joints along the chain and the parent joint of the base link are included in the group-->
-    <!--SUBGROUPS: Groups can also be formed by referencing to already defined group names-->
+<robot name="pal_sea_arm"
+    xmlns:xacro="http://ros.org/wiki/xacro">
+    <xacro:arg name="end_effector" default="pal-pro-gripper" />
+    <xacro:arg name="ft_sensor" default="no-ft-sensor" />
+    <xacro:property name="end_effector" value="$(arg end_effector)" />
+    <xacro:property name="ft_sensor" value="$(arg ft_sensor)" />
+    <xacro:property name="has_ft_sensor" value="${ft_sensor not in ['no-ft-sensor']}" />
+    <xacro:property name="robot" value="pal_sea_arm" />
+    <xacro:property name="end_effector_arg" value="${end_effector}" />
+    <xacro:if value="${end_effector_arg == 'no-end-effector'}">
+        <xacro:property name="end_effector_arg" value="no-ee" />
+    </xacro:if>
+    <!--GROUPS:
+    Representation of a set of joints and links. This can be useful for specifying DOF to plan for,
+    defining arms, end effectors, etc-->
+    <!--LINKS:
+    When a link is specified, the parent joint of that link (if it exists) is automatically
+    included-->
+    <!--JOINTS:
+    When a joint is specified, the child link of that joint (which will always exist) is
+    automatically included-->
+    <!--CHAINS:
+    When a chain is specified, all the links along the chain (including endpoints) are included in
+    the group. Additionally, all the joints that are parents to included links are also included.
+    This means that joints along the chain and the parent joint of the base link are included in the
+    group-->
+    <!--SUBGROUPS:
+    Groups can also be formed by referencing to already defined group names-->
     <group name="arm">
         <joint name="arm_1_joint" />
@@ -26,11 +43,14 @@
         <joint name="arm_tool_joint" />
     </group>
-    <xacro:include filename="$(find pal_sea_arm_moveit_config)/config/srdf/end_effectors/${end_effector}.srdf.xacro" />
-    <xacro:define_end_effector arm="arm" name="${end_effector_name}"/>
+    <xacro:include
+        filename="$(find pal_sea_arm_moveit_config)/config/srdf/end_effectors/${end_effector}.srdf.xacro" />
+    <xacro:define_end_effector arm="arm" name="${end_effector_name}" />
     <xacro:if value="${has_ft_sensor}">
-        <xacro:include filename="$(find pal_sea_arm_moveit_config)/config/srdf/disable_collisions/${robot}_${end_effector}_${ft_sensor}.srdf.xacro" />
+        <xacro:include
+            filename="$(find pal_sea_arm_moveit_config)/config/srdf/disable_collisions/${robot}_${end_effector_arg}_${ft_sensor}.srdf.xacro" />
     </xacro:if>
     <xacro:unless value="${has_ft_sensor}">
-        <xacro:include filename="$(find pal_sea_arm_moveit_config)/config/srdf/disable_collisions/${robot}_${end_effector}.srdf.xacro" />
+        <xacro:include
+            filename="$(find pal_sea_arm_moveit_config)/config/srdf/disable_collisions/${robot}_${end_effector_arg}.srdf.xacro" />
     </xacro:unless>
 </robot>
