Commit message: Add coupler link on disable collision for allegro

File: config/srdf/end_effectors/allegro-hand.srdf.xacro (robot description, xacro)
@@ -4,4 +4,6 @@
     <xacro:macro name="define_end_effector" params="arm name">
         <group name="gripper_${side}">
+              <joint name="gripper_${side}_coupler_joint"/>
+              <joint name="gripper_${side}_tc_joint"/>
               <joint name="gripper_${side}_palm_joint"/>
               <joint name="gripper_${side}_finger_1_rotatory_joint"/>
